File: board/kicad_project/hw_hacker.kicad_pcb (KiCad board)
At the start: 2 copper layers, 84 parts, among them IC1 RP2040, IC2 ME6211C33M5G-N, J1 USB_B_Mini, J2 Conn_01x06, J3 Conn_01x12, J4 Conn_01x07, J5 Conn_01x07, J6 Conn_01x02, SW1 SW_Push, U1 ATtiny84A-SS, U2 AMS1117-3.3, U3 W25Q128JVS, U4 74LS07, U5 74LS07, Y1 12MHz Crystal

Commit message: Initial board design
Parts:
- removed the R24 at (97.5, 25.9)
- removed the U2 at (28.3, 62.0)
- added H1: MountingHole, MountingHole:MountingHole_3.2mm_M3, F.Cu at (108.0, 69.8)
- added H2: MountingHole, MountingHole:MountingHole_3.2mm_M3, F.Cu at (108.0, 133.3)
- added H3: MountingHole, MountingHole:MountingHole_3.2mm_M3, F.Cu at (196.8, 69.8)
- added H4: MountingHole, MountingHole:MountingHole_3.2mm_M3, F.Cu at (196.8, 133.3)
- added IC2: ME6211C33M5G-N, Package_TO_SOT_SMD:SOT-23-5, F.Cu at (148.6, 69.8)
- added J7: Conn_01x02, Connector_PinHeader_2.54mm:PinHeader_1x02_P2.54mm_Vertical, F.Cu at (108.0, 87.0)
- added R1: 1k, Resistor_SMD:R_0402_1005Metric, F.Cu at (126.1, 108.0)
- added R25: 470R, Resistor_SMD:R_0805_2012Metric, F.Cu at (186.1, 118.1)
- C1, C10, C11, C12, C13, C2, C3, C4, C7, C8, C9: footprint Capacitor_SMD:C_0603_1608Metric -> Capacitor_SMD:C_0402_1005Metric
- C14, C16, C18, C19, C20, C21, C5, C6: footprint Capacitor_SMD:C_0603_1608Metric -> Capacitor_SMD:C_0805_2012Metric
- C15, C17: value 10u -> 1u
- IC1: footprint RP2040:QFN40P700X700X90-57N-D -> RP2040:RP2040-QFN-56
- J3: value Conn_01x12 -> Conn_01x06; footprint Connector_PinHeader_2.54mm:PinHeader_1x12_P2.54mm_Vertical -> Connector_PinHeader_2.54mm:PinHeader_1x06_P2.54mm_Vertical
- J4: value Conn_01x07 -> Conn_01x06; footprint Connector_PinHeader_2.54mm:PinHeader_1x07_P2.54mm_Vertical -> Connector_PinHeader_2.54mm:PinHeader_1x06_P2.54mm_Vertical
- J6: value Conn_01x02 -> Conn_01x07; footprint Connector_PinHeader_2.54mm:PinHeader_1x02_P2.54mm_Vertical -> Connector_PinHeader_2.54mm:PinHeader_1x07_P2.54mm_Vertical
- R10: renamed from R9; footprint Resistor_SMD:R_0603_1608Metric -> Resistor_SMD:R_0402_1005Metric
- R11: renamed from R10; footprint Resistor_SMD:R_0603_1608Metric -> Resistor_SMD:R_0402_1005Metric
- R20: renamed from R19; value 1k -> 2.2k
- R21: renamed from R20; footprint Resistor_SMD:R_0603_1608Metric -> Resistor_SMD:R_0805_2012Metric
- R22: renamed from R21; footprint Resistor_SMD:R_0603_1608Metric -> Resistor_SMD:R_0805_2012Metric
- R23: renamed from R22; footprint Resistor_SMD:R_0603_1608Metric -> Resistor_SMD:R_0805_2012Metric
- R24: renamed from R23; footprint Resistor_SMD:R_0603_1608Metric -> Resistor_SMD:R_0805_2012Metric
- R26: renamed from R25; footprint Resistor_SMD:R_0603_1608Metric -> Resistor_SMD:R_0805_2012Metric
- R27: renamed from R26; footprint Resistor_SMD:R_0603_1608Metric -> Resistor_SMD:R_0805_2012Metric
- R28: renamed from R27; footprint Resistor_SMD:R_0603_1608Metric -> Resistor_SMD:R_0805_2012Metric
- R29: renamed from R28; footprint Resistor_SMD:R_0603_1608Metric -> Resistor_SMD:R_0805_2012Metric
- R30: renamed from R29; footprint Resistor_SMD:R_0603_1608Metric -> Resistor_SMD:R_0805_2012Metric
- R31: renamed from R30; footprint Resistor_SMD:R_0603_1608Metric -> Resistor_SMD:R_0805_2012Metric
- R32: renamed from R31; footprint Resistor_SMD:R_0603_1608Metric -> Resistor_SMD:R_0805_2012Metric
- R33: renamed from R32; footprint Resistor_SMD:R_0603_1608Metric -> Resistor_SMD:R_0805_2012Metric
- R34: renamed from R33; footprint Resistor_SMD:R_0603_1608Metric -> Resistor_SMD:R_0805_2012Metric
- R35: renamed from R34; footprint Resistor_SMD:R_0603_1608Metric -> Resistor_SMD:R_0805_2012Metric
- SW1: footprint Button_Switch_SMD:SW_Push_1P1T_NO_6x6mm_H9.5mm -> Button_Switch_SMD:SW_SPST_SKQG_WithStem
- Y1: value 12MHz Crystal -> X322512MSB4SI 12MHz; footprint YSX321SL:YSX321SL -> Crystal:Crystal_SMD_3225-4Pin_3.2x2.5mm
- moved R5 169.3 mm to (186.1, 108.5)
- moved R7 167.8 mm to (186.1, 106.7)
- moved R16 166.2 mm to (186.1, 110.2)
- moved R3 164.6 mm to (186.1, 99.1)
- moved R12 161.1 mm to (186.1, 96.5)
- moved R4 159.8 mm to (186.1, 103.1)
- moved R14 157.0 mm to (186.1, 104.9)
- moved R13 156.5 mm to (186.1, 101.3)
- moved R18 156.1 mm to (172.1, 104.1), turned to 180 degrees
- moved R15 154.0 mm to (172.1, 107.7), turned to 180 degrees
- moved R19 150.9 mm to (172.1, 96.5), turned to 180 degrees
- moved R6 150.1 mm to (172.1, 105.9), turned to 180 degrees
- moved R8 146.1 mm to (172.1, 99.1), turned to 180 degrees
- moved SW1 143.8 mm to (143.5, 118.7), turned to 180 degrees
- moved D6 143.4 mm to (194.3, 104.1), turned to 180 degrees
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- renumbered IC2 to IC3, R11 to R12, R12 to R13, R13 to R14, R14 to R15, R15 to R16, R16 to R17, R17 to R18, R18 to R19, R1 to R2, R2 to R3, R3 to R4, R4 to R5, R5 to R6, R6 to R7, R7 to R8, R8 to R9, U3 to U2, U4 to U3, U5 to U4
Connections:
- net Net-(C3-Pad1) renamed /RP2040 Attacker/1V1
- C16 pad 1: /Power/AVR_PWR_CE -> /Power/USB_VBUS
- IC1 pad 21: Net-(C2-Pad1) -> Net-(IC1-Pad21)
- J2 pad 4: GND -> /RP2040 Attacker/SWCLK
- J2 pad 6: /RP2040 Attacker/SWCLK -> GND
- J3 pad 2: /Indicator LEDs/RP2040_3V3 -> /RP2040 Attacker/GPIO29
- J3 pad 3: GND -> /RP2040 Attacker/GPIO28
- J3 pad 4: GND -> /RP2040 Attacker/GPIO27
- J3 pad 5: /RP2040 Attacker/GPIO12 -> /RP2040 Attacker/GPIO26
- J3 pad 6: /RP2040 Attacker/GPIO13 -> GND
- J4 pad 1: GND -> /Indicator LEDs/RP2040_3V3
- J4 pad 2: /AVR Target/AVR_PA0 -> /RP2040 Attacker/GPIO12
- J4 pad 3: /AVR Target/AVR_PA1 -> /RP2040 Attacker/GPIO13
- J4 pad 4: /AVR Target/AVR_PA2 -> /RP2040 Attacker/GPIO14
- J4 pad 5: /AVR Target/AVR_PA3 -> /RP2040 Attacker/GPIO15
- J4 pad 6: /AVR Target/AVR_PA4 -> GND
- J5 pad 1: /AVR Target/AVR_PA6 -> GND
- J5 pad 2: /AVR Target/AVR_PA7 -> /AVR Target/AVR_PA0
- J5 pad 3: /AVR Target/AVR_PB2 -> /AVR Target/AVR_PA1
- J5 pad 4: /AVR Target/AVR_PB3 -> /AVR Target/AVR_PA2
- J5 pad 5: /AVR Target/AVR_PB1 -> /AVR Target/AVR_PA3
- J5 pad 6: /AVR Target/AVR_PB0 -> /AVR Target/AVR_PA4
- J5 pad 7: /AVR Target/AVR_3V3 -> /AVR Target/AVR_PA5
- J6 pad 1: GND -> /AVR Target/AVR_3V3
- J6 pad 2: /RP2040 Attacker/QSPI Flash/~{USB_BOOT} -> /AVR Target/AVR_PB0
- R22 pad 1: Net-(R21-Pad1) -> Net-(R22-Pad1)
- R23 pad 1: Net-(R22-Pad1) -> Net-(R23-Pad1)
- R24 pad 1: Net-(R23-Pad1) -> Net-(R24-Pad1)
- R26 pad 1: Net-(R25-Pad1) -> Net-(R26-Pad1)
- R27 pad 1: Net-(R26-Pad1) -> Net-(R27-Pad1)
- R28 pad 1: Net-(R27-Pad1) -> Net-(R28-Pad1)
- R29 pad 1: Net-(R28-Pad1) -> Net-(R29-Pad1)
- R30 pad 1: Net-(R29-Pad1) -> Net-(R30-Pad1)
- R31 pad 1: Net-(R30-Pad1) -> Net-(R31-Pad1)
- R32 pad 1: Net-(R31-Pad1) -> Net-(R32-Pad1)
- R33 pad 1: Net-(R32-Pad1) -> Net-(R33-Pad1)
- U3 pad 1: /AVR Target/AVR_PA0 -> /AVR Target/AVR_PB3
- U3 pad 10: Net-(R25-Pad1) -> Net-(R23-Pad1)
- U3 pad 11: /AVR Target/AVR_PA4 -> /AVR Target/AVR_PA1
- U3 pad 12: Net-(R26-Pad1) -> Net-(R24-Pad1)
- U3 pad 13: /AVR Target/AVR_PA5 -> /AVR Target/AVR_PA2
- U3 pad 2: Net-(R21-Pad1) -> Net-(R33-Pad1)
- U3 pad 3: /AVR Target/AVR_PA1 -> /AVR Target/AVR_PB1
- U3 pad 4: Net-(R22-Pad1) -> Net-(R31-Pad1)
- U3 pad 5: /AVR Target/AVR_PA2 -> /AVR Target/AVR_PB0
- U3 pad 6: Net-(R23-Pad1) -> Net-(R30-Pad1)
- U3 pad 8: Net-(R24-Pad1) -> Net-(R22-Pad1)
- U3 pad 9: /AVR Target/AVR_PA3 -> /AVR Target/AVR_PA0
- U4 pad 1: /AVR Target/AVR_PA6 -> /AVR Target/AVR_PA3
- U4 pad 10: Net-(R31-Pad1) -> Net-(R29-Pad1)
- U4 pad 11: /AVR Target/AVR_PB2 -> /AVR Target/AVR_PA7
- U4 pad 13: /AVR Target/AVR_PB3 -> /AVR Target/AVR_PB2
- U4 pad 2: Net-(R27-Pad1) -> Net-(R25-Pad1)
- U4 pad 3: /AVR Target/AVR_PA7 -> /AVR Target/AVR_PA4
- U4 pad 4: Net-(R28-Pad1) -> Net-(R26-Pad1)
- U4 pad 5: /AVR Target/AVR_PB0 -> /AVR Target/AVR_PA5
- U4 pad 6: Net-(R29-Pad1) -> Net-(R27-Pad1)
- U4 pad 8: Net-(R30-Pad1) -> Net-(R28-Pad1)
- U4 pad 9: /AVR Target/AVR_PB1 -> /AVR Target/AVR_PA6
Routing:
- net GND: track 0.00 -> 159.4 mm, vias 0 -> 35
- net Net-(IC1-Pad4): track 0.00 -> 84.6 mm, vias 0 -> 2
- net Net-(IC1-Pad5): track 0.00 -> 82.4 mm, vias 0 -> 2
- net Net-(IC1-Pad9): track 0.00 -> 82.3 mm, vias 0 -> 2
- net Net-(IC1-Pad6): track 0.00 -> 81.7 mm, vias 0 -> 2
- net /Power/AVR_PWR_CE: track 0.00 -> 80.9 mm, vias 0 -> 2
- net Net-(IC1-Pad7): track 0.00 -> 80.8 mm, vias 0 -> 2
- net Net-(IC1-Pad8): track 0.00 -> 80.7 mm, vias 0 -> 2
- net /Indicator LEDs/RP2040_3V3: track 0.00 -> 72.7 mm, vias 0 -> 4
- net Net-(IC1-Pad11): track 0.00 -> 70.3 mm, vias 0 -> 2
- net Net-(IC1-Pad12): track 0.00 -> 70.3 mm, vias 0 -> 2
- net Net-(IC1-Pad28): track 0.00 -> 63.9 mm, vias 0 -> 2
- net Net-(IC1-Pad27): track 0.00 -> 59.8 mm, vias 0 -> 2
- net Net-(IC1-Pad35): track 0.00 -> 51.2 mm, vias 0 -> 2
- net /AVR Target/AVR_3V3: track 0.00 -> 51.2 mm, vias 0 -> 1
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- added copper zone on F.Cu, net /Indicator LEDs/RP2040_3V3
- added copper zone on B.Cu, net GND
Other:
- board outline added: 101.6 x 76.2 mm
- board text added: "3V3"
- board text added: "ADC0"
- board text added: "ADC1"
- board text added: "ADC2"
- board text added: "ADC3"
- board text added: "AVR 3V3"
- board text added: "AVR PWR"
- board text added: "AVR Target"
- board text added: "BOOTSEL"
- board text added: "CLK/PB0"
- board text added: "GND"
- board text added: "IO12"
- board text added: "IO13"
- board text added: "IO14"
- board text added: "IO15"
- board text added: "PA0"
- board text added: "PA1"
- board text added: "PA2"
- board text added: "PA3"
- board text added: "PA4"
- board text added: "PA5"
- board text added: "PA6"
- board text added: "PA7"
- board text added: "PB1"
- board text added: "PB2"
- board text added: "RP2040 Attacker"
- board text added: "RP2040 PWR"
- board text added: "Reset"
- board text added: "SER RX"
- board text added: "SER TX"
- board text added: "SWCLK"
- board text added: "SWDIO"
- board text added: "~{RST}/PB3"
