File: board/kicad_project/hw_hacker.kicad_pcb (KiCad board)
At the start: 2 copper layers, 101.6 x 76.2 mm, 90 parts, among them IC1 RP2040, IC2 ME6211C33M5G-N, IC3 ME6211C33M5G-N, J1 USB_B_Mini, J2 Conn_01x06, J3 Conn_01x06, J4 Conn_01x06, J5 Conn_01x07, J6 Conn_01x07, J7 Conn_01x02, SW1 SW_Push, U1 ATtiny84A-SS, U2 W25Q128JVS, U3 74LS07, U4 74LS07, Y1 X322512MSB4SI 12MHz

Commit message: Add LCSC part numbers to board file
* Also replaced flash chip with cheaper/smaller HG25Q16 that should be
  pin compatible
Parts:
- U2: value W25Q128JVS -> HG25Q16
- U3, U4: value 74LS07 -> 74HC07
