File: board/kicad_project/attacker.kicad_sch (KiCad schematic)
At the start: 36 parts, among them IC1 RP2040, J2 Conn_01x06, J3 Conn_01x12, SW1 SW_Push, Y1 12MHz Crystal

Commit message: Initial board design
Parts:
- removed J3: Conn_01x12, Connector_PinHeader_2.54mm:PinHeader_1x12_P2.54mm_Vertical, symbol Connector_Generic:Conn_01x12
- removed Y1: 12MHz Crystal, YSX321SL:YSX321SL, symbol Device:Crystal_GND2
- added J3, J4: Conn_01x06, Connector_PinHeader_2.54mm:PinHeader_1x06_P2.54mm_Vertical, symbol Connector_Generic:Conn_01x06
- added R1: 1k, Resistor_SMD:R_0402_1005Metric, symbol Device:R
- added Y1: X322512MSB4SI 12MHz, Crystal:Crystal_SMD_3225-4Pin_3.2x2.5mm, symbol Device:Crystal_GND24
- C1, C10, C11, C12, C13, C2, C3, C4, C7, C8, C9: footprint Capacitor_SMD:C_0603_1608Metric -> Capacitor_SMD:C_0402_1005Metric
- C5, C6: footprint Capacitor_SMD:C_0603_1608Metric -> Capacitor_SMD:C_0805_2012Metric
- IC1: footprint RP2040:QFN40P700X700X90-57N-D -> RP2040:RP2040-QFN-56
- R10: renamed from R9; footprint Resistor_SMD:R_0603_1608Metric -> Resistor_SMD:R_0402_1005Metric
- R11: renamed from R10; footprint Resistor_SMD:R_0603_1608Metric -> Resistor_SMD:R_0402_1005Metric
- SW1: footprint Button_Switch_SMD:SW_Push_1P1T_NO_6x6mm_H9.5mm -> Button_Switch_SMD:SW_SPST_SKQG_WithStem
- renumbered R11 to R12, R12 to R13, R13 to R14, R14 to R15, R15 to R16, R16 to R17, R17 to R18, R18 to R19, R1 to R2, R2 to R3, R3 to R4, R4 to R5, R5 to R6, R6 to R7, R7 to R8, R8 to R9
Connections:
- net 3V3: now also J3.1 (Pin_1), J4.1 (Pin_1)
- net GND: now also J2.6 (Pin_6), J3.6 (Pin_6), J4.6 (Pin_6), Y1.2, Y1.4; no longer J2.4 (Pin_4)
- net GPIO12: now also J4.2 (Pin_2)
- net GPIO13: now also J4.3 (Pin_3)
- net GPIO14: now also J4.4 (Pin_4)
- net GPIO15: now also J4.5 (Pin_5)
- net GPIO26: now also J3.5 (Pin_5)
- net GPIO27: now also J3.4 (Pin_4)
- net GPIO28: now also J3.3 (Pin_3)
- net GPIO29: now also J3.2 (Pin_2)
- net SWCLK: now also J2.4 (Pin_4); no longer J2.6 (Pin_6)
- net at C2.1: now also R1.2, Y1.1; no longer IC1.21 (XOUT)
- net at C1.1, IC1.20 (XIN): now also Y1.3
- net 1V1: now reaches C3.1, C4.1, C5.1, IC1.23 (DVDD_1), IC1.45 (VREG_VOUT), IC1.50 (DVDD_2)
- new net: IC1.21 (XOUT), R1.1
Other:
- note added: "ADC Header"
- note added: "AVR pin uses (from AVR perspective) PA4: SPI CLK/I2C SCL PA5: SPI CIPO (TX from AVR) PA6: SPI COPI (RX to AVR)/I2C SDA PB0: CLK Input PB3: RESET_N/debugWire IO"
- note added: "Connections to use by signal type (RP2040 perspective): Clock: GPIO21-PB0 ~{Reset}: GPIO24-PB3 SPI: GPIO6-PA4 (SPI0 SCLK) GPIO16-PA5 (SPI0 RX) GPIO19-PA6 (SPI0 TX) I2C: GPIO8-PA6 (I2C0 SDA) GPIO17-PA4 (I2C0 SCL) UART: GPIO4-PA2 or GPIO8-PA6 or GPIO20-PB1 (UART1 TX) GPIO5-PA3 or GPIO9-PA7 or GPIO21-PB2 (UART1 RX)"
- note removed: "AVR pin uses (from AVR perspective) PA4: SPI CLK/I2C SCL PA5: SPI MISO (TX from AVR) PA6: SPI MOSI (RX to AVR)/I2C SDA PB0: CLK Input PB3: RESET_N/debugWire IO"
- note removed: "Connections to use by signal type (RP2040 perspective): Clock: GPIO21-PB0 SPI: GPIO6-PA4 (SPI0 SCLK) GPIO16-PA5 (SPI0 RX) GPIO19-PA6 (SPI0 TX) I2C: GPIO8-PA6 (I2C0 SDA) GPIO17-PA4 (I2C0 SCL) UART: GPIO4-PA2 or GPIO8-PA6 or GPIO20-PB1 (UART1 TX) GPIO5-PA3 or GPIO9-PA7 or GPIO21-PB2 (UART1 RX)"
- moved on the sheet: C1, C2

Commit message: Added lcsc part numbers
Parts:
- C1, C2: LCSC Part (none) -> C1557
- C10, C11, C12, C13, C3, C4, C7, C8, C9: LCSC Part (none) -> C1525
- C5, C6: LCSC Part (none) -> C28323
- IC1: LCSC Part (none) -> C2040
- J2, J3, J4: JLCPCB BOM (none) -> 0
- R1: LCSC Part (none) -> C11702
- R10, R11: LCSC Part (none) -> C172043
- R12, R13, R14, R15, R16, R17, R18, R19, R2, R3, R4, R5, R6, R7, R8, R9: LCSC Part (none) -> C4190
- SW1: LCSC Part (none) -> C318884
- Y1: LCSC Part (none) -> C9002
Changed lines of the file:
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@@
+      (effects (font (size 1.27 1.27)) hide)
+    )
+    (property "LCSC Part" "C11702" (id 4) (at 58.42 96.52 0)
       (effects (font (size 1.27 1.27)) hide)
     )
@@
       (effects (font (size 1.27 1.27)) hide)
     )
+    (property "LCSC Part" "C4190" (id 4) (at 69.85 106.68 0)
+      (effects (font (size 1.27 1.27)) hide)
+    )
     (pin "1")
     (pin "2")
@@
       (effects (font (size 1.27 1.27)) hide)
     )
+    (property "LCSC Part" "C4190" (id 4) (at 154.94 69.85 0)
+      (effects (font (size 1.27 1.27)) hide)
+    )
     (pin "1")
     (pin "2")
@@
       (effects (font (size 1.27 1.27)) hide)
     )
+    (property "LCSC Part" "C4190" (id 4) (at 154.94 74.93 0)
+      (effects (font (size 1.27 1.27)) hide)
+    )
     (pin "1")
     (pin "2")
@@
       (effects (font (size 1.27 1.27)) hide)
     )
+    (property "LCSC Part" "C4190" (id 4) (at 154.94 80.01 0)
+      (effects (font (size 1.27 1.27)) hide)
+    )
     (pin "1")
     (pin "2")
@@
       (effects (font (size 1.27 1.27)) hide)
     )
+    (property "LCSC Part" "C4190" (id 4) (at 154.94 85.09 0)
+      (effects (font (size 1.27 1.27)) hide)
+    )
     (pin "1")
     (pin "2")
@@
       (effects (font (size 1.27 1.27)) hide)
     )
+    (property "LCSC Part" "C4190" (id 4) (at 154.94 105.41 0)
+      (effects (font (size 1.27 1.27)) hide)
+    )
     (pin "1")
     (pin "2")
@@
       (effects (font (size 1.27 1.27)) hide)
     )
+    (property "LCSC Part" "C4190" (id 4) (at 154.94 113.03 0)
+      (effects (font (size 1.27 1.27)) hide)
+    )
     (pin "1")
     (pin "2")
@@
       (effects (font (size 1.27 1.27)) hide)
     )
+    (property "LCSC Part" "C4190" (id 4) (at 154.94 123.19 0)
+      (effects (font (size 1.27 1.27)) hide)
+    )
     (pin "1")
     (pin "2")
@@
       (effects (font (size 1.27 1.27)) hide)
     )
+    (property "LCSC Part" "C172043" (id 4) (at 156.21 49.53 0)
+      (effects (font (size 1.27 1.27)) hide)
+    )
     (pin "1")
     (pin "2")
@@
       (effects (font (size 1.27 1.27)) hide)
     )
+    (property "LCSC Part" "C172043" (id 4) (at 156.21 57.15 0)
+      (effects (font (size 1.27 1.27)) hide)
+    )
     (pin "1")
     (pin "2")
@@
       (effects (font (size 1.27 1.27)) hide)
     )
+    (property "LCSC Part" "C4190" (id 4) (at 168.91 67.31 0)
+      (effects (font (size 1.27 1.27)) hide)
+    )
     (pin "1")
     (pin "2")
@@
       (effects (font (size 1.27 1.27)) hide)
     )
+    (property "LCSC Part" "C4190" (id 4) (at 168.91 72.39 0)
+      (effects (font (size 1.27 1.27)) hide)
+    )
     (pin "1")
     (pin "2")
@@
       (effects (font (size 1.27 1.27)) hide)
     )
+    (property "LCSC Part" "C4190" (id 4) (at 168.91 77.47 0)
+      (effects (font (size 1.27 1.27)) hide)
+    )
     (pin "1")
     (pin "2")
@@
       (effects (font (size 1.27 1.27)) hide)
     )
+    (property "LCSC Part" "C4190" (id 4) (at 168.91 82.55 0)
+      (effects (font (size 1.27 1.27)) hide)
+    )
     (pin "1")
     (pin "2")
@@
       (effects (font (size 1.27 1.27)) hide)
     )
+    (property "LCSC Part" "C4190" (id 4) (at 168.91 102.87 0)
+      (effects (font (size 1.27 1.27)) hide)
+    )
     (pin "1")
     (pin "2")
@@
       (effects (font (size 1.27 1.27)) hide)
     )
+    (property "LCSC Part" "C4190" (id 4) (at 168.91 110.49 0)
+      (effects (font (size 1.27 1.27)) hide)
+    )
     (pin "1")
     (pin "2")
@@
       (effects (font (size 1.27 1.27)) hide)
     )
+    (property "LCSC Part" "C4190" (id 4) (at 168.91 115.57 0)
+      (effects (font (size 1.27 1.27)) hide)
+    )
     (pin "1")
     (pin "2")
@@
       (effects (font (size 1.27 1.27)) hide)
     )
+    (property "LCSC Part" "C4190" (id 4) (at 168.91 120.65 0)
+      (effects (font (size 1.27 1.27)) hide)
+    )
     (pin "1")
     (pin "2")
@@
       (effects (font (size 1.27 1.27)) hide)
     )
+    (property "LCSC Part" "C1557" (id 4) (at 33.02 86.36 0)
+      (effects (font (size 1.27 1.27)) hide)
+    )
     (pin "1")
     (pin "2")
@@
       (effects (font (size 1.27 1.27)) hide)
     )
+    (property "LCSC Part" "C1557" (id 4) (at 33.02 96.52 0)
+      (effects (font (size 1.27 1.27)) hide)
+    )
     (pin "1")
     (pin "2")
@@
       (effects (font (size 1.27 1.27)) hide)
     )
+    (property "LCSC Part" "C1525" (id 4) (at 60.96 46.99 0)
+      (effects (font (size 1.27 1.27)) hide)
+    )
     (pin "1")
     (pin "2")
@@
       (effects (font (size 1.27 1.27)) hide)
     )
+    (property "LCSC Part" "C1525" (id 4) (at 72.39 46.99 0)
+      (effects (font (size 1.27 1.27)) hide)
+    )
     (pin "1")
     (pin "2")
@@
       (effects (font (size 1.27 1.27)) hide)
     )
+    (property "LCSC Part" "C28323" (id 4) (at 83.82 46.99 0)
+      (effects (font (size 1.27 1.27)) hide)
+    )
     (pin "1")
     (pin "2")
@@
       (effects (font (size 1.27 1.27)) hide)
     )
+    (property "LCSC Part" "C28323" (id 4) (at 133.35 34.29 0)
+      (effects (font (size 1.27 1.27)) hide)
+    )
     (pin "1")
     (pin "2")
@@
       (effects (font (size 1.27 1.27)) hide)
     )
+    (property "LCSC Part" "C1525" (id 4) (at 143.51 34.29 0)
+      (effects (font (size 1.27 1.27)) hide)
+    )
     (pin "1")
     (pin "2")
@@
       (effects (font (size 1.27 1.27)) hide)
     )
+    (property "LCSC Part" "C1525" (id 4) (at 154.94 34.29 0)
+      (effects (font (size 1.27 1.27)) hide)
+    )
     (pin "1")
     (pin "2")
@@
       (effects (font (size 1.27 1.27)) hide)
     )
+    (property "LCSC Part" "C1525" (id 4) (at 166.37 34.29 0)
+      (effects (font (size 1.27 1.27)) hide)
+    )
     (pin "1")
     (pin "2")
@@
       (effects (font (size 1.27 1.27)) hide)
     )
+    (property "LCSC Part" "C1525" (id 4) (at 177.8 34.29 0)
+      (effects (font (size 1.27 1.27)) hide)
+    )
     (pin "1")
     (pin "2")
@@
       (effects (font (size 1.27 1.27)) hide)
     )
+    (property "LCSC Part" "C1525" (id 4) (at 189.23 34.29 0)
+      (effects (font (size 1.27 1.27)) hide)
+    )
     (pin "1")
     (pin "2")
@@
       (effects (font (size 1.27 1.27)) hide)
     )
+    (property "LCSC Part" "C1525" (id 4) (at 200.66 34.29 0)
+      (effects (font (size 1.27 1.27)) hide)
+    )
     (pin "1")
     (pin "2")
@@
     )
     (property "Datasheet" "~" (id 3) (at 212.09 34.29 0)
+      (effects (font (size 1.27 1.27)) hide)
+    )
+    (property "LCSC Part" "C1525" (id 4) (at 212.09 34.29 0)
       (effects (font (size 1.27 1.27)) hide)
     )
@@
       (effects (font (size 1.27 1.27)) hide)
     )
+    (property "LCSC Part" "C318884" (id 4) (at 69.85 120.65 0)
+      (effects (font (size 1.27 1.27)) hide)
+    )
     (pin "1")
     (pin "2")
@@
       (effects (font (size 1.27 1.27)) hide)
     )
+    (property "LCSC Part" "C9002" (id 4) (at 46.99 91.44 0)
+      (effects (font (size 1.27 1.27)) hide)
+    )
     (pin "1")
     (pin "2")
@@
     )
     (property "Datasheet" "~" (id 3) (at 53.34 132.08 0)
+      (effects (font (size 1.27 1.27)) hide)
+    )
+    (property "JLCPCB BOM" "0" (id 4) (at 53.34 132.08 0)
       (effects (font (size 1.27 1.27)) hide)
     )
@@
       (effects (font (size 1.27 1.27)) hide)
     )
+    (property "JLCPCB BOM" "0" (id 4) (at 115.57 170.18 0)
+      (effects (font (size 1.27 1.27)) hide)
+    )
     (pin "1")
     (pin "2")
@@
       (effects (font (size 1.27 1.27)) hide)
     )
+    (property "JLCPCB BOM" "0" (id 4) (at 153.67 170.18 0)
+      (effects (font (size 1.27 1.27)) hide)
+    )
     (pin "1")
     (pin "2")
@@
       (effects (font (size 1.27 1.27)) (justify left) hide)
     )
-    (pin "1")
+    (property "LCSC Part" "C2040" (id 12) (at 114.3 95.25 0)
+      (effects (font (size 1.27 1.27)) hide)
+    )
+    (pin "1")
