File: board/kicad_project/flash.kicad_sch (KiCad schematic)
At the start: 5 parts, among them J6 Conn_01x02, U3 W25Q128JVS

Commit message: Initial board design
Parts:
- C19: footprint Capacitor_SMD:C_0603_1608Metric -> Capacitor_SMD:C_0805_2012Metric
- R20: renamed from R19; value 1k -> 2.2k
- R21: renamed from R20; footprint Resistor_SMD:R_0603_1608Metric -> Resistor_SMD:R_0805_2012Metric
- renumbered J6 to J7, U3 to U2
Connections:
- net GND: now also J7.2 (Pin_2); no longer J7.1 (Pin_1)
- net ~{USB_BOOT}: now also J7.1 (Pin_1); no longer J7.2 (Pin_2)
Other:
- moved on the sheet: J7
Changed lines of the file:
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@@
   (symbol (lib_id "power:GND") (at 109.22 76.2 0) (unit 1)
     (in_bom yes) (on_board yes)
-    (property "Reference" "#PWR015" (id 0) (at 109.22 82.55 0)
+    (property "Reference" "#PWR020" (id 0) (at 109.22 82.55 0)
       (effects (font (size 1.27 1.27)) hide)
     )
@@
   (symbol (lib_id "power:GND") (at 139.7 106.68 0) (unit 1)
     (in_bom yes) (on_board yes) (fields_autoplaced)
-    (property "Reference" "#PWR016" (id 0) (at 139.7 113.03 0)
+    (property "Reference" "#PWR021" (id 0) (at 139.7 113.03 0)
       (effects (font (size 1.27 1.27)) hide)
     )
@@
   (symbol (lib_id "power:GND") (at 144.78 81.28 0) (unit 1)
     (in_bom yes) (on_board yes)
-    (property "Reference" "#PWR017" (id 0) (at 144.78 87.63 0)
+    (property "Reference" "#PWR022" (id 0) (at 144.78 87.63 0)
       (effects (font (size 1.27 1.27)) hide)
     )
@@
   (symbol (lib_id "Device:R") (at 111.76 85.09 0) (unit 1)
     (in_bom yes) (on_board yes) (fields_autoplaced)
-    (property "Reference" "R19" (id 0) (at 114.3 83.8199 0)
+    (property "Reference" "R20" (id 0) (at 114.3 83.8199 0)
       (effects (font (size 1.27 1.27)) (justify left))
     )
-    (property "Value" "1k" (id 1) (at 114.3 86.3599 0)
+    (property "Value" "2.2k" (id 1) (at 114.3 86.3599 0)
       (effects (font (size 1.27 1.27)) (justify left))
     )
@@
   (symbol (lib_id "Device:R") (at 121.92 85.09 0) (unit 1)
     (in_bom yes) (on_board yes) (fields_autoplaced)
-    (property "Reference" "R20" (id 0) (at 124.46 83.8199 0)
+    (property "Reference" "R21" (id 0) (at 124.46 83.8199 0)
       (effects (font (size 1.27 1.27)) (justify left))
     )
@@
       (effects (font (size 1.27 1.27)) (justify left))
     )
-    (property "Footprint" "Resistor_SMD:R_0603_1608Metric" (id 2) (at 120.142 85.09 90)
+    (property "Footprint" "Resistor_SMD:R_0805_2012Metric" (id 2) (at 120.142 85.09 90)
       (effects (font (size 1.27 1.27)) hide)
     )
@@
     (pin "2")
   )
-  (symbol (lib_id "Connector_Generic:Conn_01x02") (at 109.22 68.58 90) (unit 1)
+  (symbol (lib_id "Connector_Generic:Conn_01x02") (at 111.76 68.58 270) (mirror x) (unit 1)
     (in_bom yes) (on_board yes) (fields_autoplaced)
-    (property "Reference" "J6" (id 0) (at 114.3 69.3419 90)
-      (effects (font (size 1.27 1.27)) (justify right))
+    (property "Reference" "J7" (id 0) (at 114.3 69.3419 90)
+      (effects (font (size 1.27 1.27)) (justify left))
     )
     (property "Value" "Conn_01x02" (id 1) (at 114.3 71.8819 90)
-      (effects (font (size 1.27 1.27)) (justify right))
+      (effects (font (size 1.27 1.27)) (justify left))
     )
-    (property "Footprint" "Connector_PinHeader_2.54mm:PinHeader_1x02_P2.54mm_Vertical" (id 2) (at 109.22 68.58 0)
+    (property "Footprint" "Connector_PinHeader_2.54mm:PinHeader_1x02_P2.54mm_Vertical" (id 2) (at 111.76 68.58 0)
       (effects (font (size 1.27 1.27)) hide)
     )
-    (property "Datasheet" "~" (id 3) (at 109.22 68.58 0)
+    (property "Datasheet" "~" (id 3) (at 111.76 68.58 0)
       (effects (font (size 1.27 1.27)) hide)
     )
@@
       (effects (font (size 1.27 1.27)) (justify left))
     )
-    (property "Footprint" "Capacitor_SMD:C_0603_1608Metric" (id 2) (at 145.7452 80.01 0)
+    (property "Footprint" "Capacitor_SMD:C_0805_2012Metric" (id 2) (at 145.7452 80.01 0)
       (effects (font (size 1.27 1.27)) hide)
     )
@@
   (symbol (lib_id "Memory_Flash:W25Q128JVS") (at 139.7 93.98 0) (unit 1)
     (in_bom yes) (on_board yes)
-    (property "Reference" "U3" (id 0) (at 154.94 81.28 0))
+    (property "Reference" "U2" (id 0) (at 154.94 81.28 0))
     (property "Value" "W25Q128JVS" (id 1) (at 154.94 83.82 0))
     (property "Footprint" "Package_SO:SOIC-8_5.23x5.23mm_P1.27mm" (id 2) (at 139.7 93.98 0)

Commit message: Added lcsc part numbers
Parts:
- C19: LCSC Part (none) -> C49678
- J7, R21: JLCPCB BOM (none) -> 0
- R20: LCSC Part (none) -> C4190
- U2: LCSC Part (none) -> C97521
Changed lines of the file:
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@@
+      (effects (font (size 1.27 1.27)) hide)
+    )
+    (property "LCSC Part" "C4190" (id 4) (at 111.76 85.09 0)
       (effects (font (size 1.27 1.27)) hide)
     )
@@
       (effects (font (size 1.27 1.27)) hide)
     )
+    (property "JLCPCB BOM" "0" (id 4) (at 121.92 85.09 0)
+      (effects (font (size 1.27 1.27)) hide)
+    )
     (pin "1")
     (pin "2")
@@
     )
     (property "Datasheet" "~" (id 3) (at 111.76 68.58 0)
+      (effects (font (size 1.27 1.27)) hide)
+    )
+    (property "JLCPCB BOM" "0" (id 4) (at 111.76 68.58 0)
       (effects (font (size 1.27 1.27)) hide)
     )
@@
       (effects (font (size 1.27 1.27)) hide)
     )
+    (property "LCSC Part" "C49678" (id 4) (at 144.78 76.2 0)
+      (effects (font (size 1.27 1.27)) hide)
+    )
     (pin "1")
     (pin "2")
@@
       (effects (font (size 1.27 1.27)) hide)
     )
+    (property "LCSC Part" "C97521" (id 4) (at 139.7 93.98 0)
+      (effects (font (size 1.27 1.27)) hide)
+    )
