File: board/kicad_project/target.kicad_sch (KiCad schematic)
At the start: 4 parts, among them J4 Conn_01x07, J5 Conn_01x07, U1 ATtiny84A-SS

Commit message: Initial board design
Parts:
- C14: footprint Capacitor_SMD:C_0603_1608Metric -> Capacitor_SMD:C_0805_2012Metric
- renumbered J4 to J5, J5 to J6
Connections:
- net AVR_3V3: now also J6.1 (Pin_1); no longer J6.7 (Pin_7)
- net AVR_PA6: now also J6.7 (Pin_7); no longer J6.1 (Pin_1)
- net AVR_PA7: now also J6.6 (Pin_6); no longer J6.2 (Pin_2)
- net AVR_PB0: now also J6.2 (Pin_2); no longer J6.6 (Pin_6)
- net AVR_PB1: now also J6.3 (Pin_3); no longer J6.5 (Pin_5)
- net AVR_PB2: now also J6.5 (Pin_5); no longer J6.3 (Pin_3)
Changed lines of the file:
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@@
   (symbol (lib_id "power:GND") (at 114.3 130.81 0) (unit 1)
     (in_bom yes) (on_board yes) (fields_autoplaced)
-    (property "Reference" "#PWR010" (id 0) (at 114.3 137.16 0)
+    (property "Reference" "#PWR013" (id 0) (at 114.3 137.16 0)
       (effects (font (size 1.27 1.27)) hide)
     )
@@
   (symbol (lib_id "power:GND") (at 119.38 81.28 0) (unit 1)
     (in_bom yes) (on_board yes)
-    (property "Reference" "#PWR011" (id 0) (at 119.38 87.63 0)
+    (property "Reference" "#PWR014" (id 0) (at 119.38 87.63 0)
       (effects (font (size 1.27 1.27)) hide)
     )
@@
   (symbol (lib_id "power:GND") (at 171.45 92.71 0) (unit 1)
     (in_bom yes) (on_board yes) (fields_autoplaced)
-    (property "Reference" "#PWR012" (id 0) (at 171.45 99.06 0)
+    (property "Reference" "#PWR015" (id 0) (at 171.45 99.06 0)
       (effects (font (size 1.27 1.27)) hide)
     )
@@
       (effects (font (size 1.27 1.27)) (justify left))
     )
-    (property "Footprint" "Capacitor_SMD:C_0603_1608Metric" (id 2) (at 120.3452 80.01 0)
+    (property "Footprint" "Capacitor_SMD:C_0805_2012Metric" (id 2) (at 120.3452 80.01 0)
       (effects (font (size 1.27 1.27)) hide)
     )
@@
   (symbol (lib_id "Connector_Generic:Conn_01x07") (at 191.77 99.06 0) (unit 1)
     (in_bom yes) (on_board yes) (fields_autoplaced)
-    (property "Reference" "J4" (id 0) (at 194.31 97.79 0)
+    (property "Reference" "J5" (id 0) (at 194.31 97.79 0)
       (effects (font (size 1.27 1.27)) (justify left))
     )
@@
     (pin "7")
   )
-  (symbol (lib_id "Connector_Generic:Conn_01x07") (at 191.77 127 0) (unit 1)
-    (in_bom yes) (on_board yes) (fields_autoplaced)
-    (property "Reference" "J5" (id 0) (at 194.31 125.73 0)
-      (effects (font (size 1.27 1.27)) (justify left))
-    )
-    (property "Value" "Conn_01x07" (id 1) (at 194.31 128.27 0)
-      (effects (font (size 1.27 1.27)) (justify left))
-    )
+  (symbol (lib_id "Connector_Generic:Conn_01x07") (at 191.77 127 0) (mirror x) (unit 1)
+    (in_bom yes) (on_board yes)
+    (property "Reference" "J6" (id 0) (at 199.898 125.73 0))
+    (property "Value" "Conn_01x07" (id 1) (at 199.898 128.27 0))
     (property "Footprint" "Connector_PinHeader_2.54mm:PinHeader_1x07_P2.54mm_Vertical" (id 2) (at 191.77 127 0)
       (effects (font (size 1.27 1.27)) hide)

Commit message: Added lcsc part numbers
Parts:
- C14: LCSC Part (none) -> C49678
- J5, J6: JLCPCB BOM (none) -> 0
- U1: LCSC Part (none) -> C14909
Changed lines of the file:
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@@
+      (effects (font (size 1.27 1.27)) hide)
+    )
+    (property "LCSC Part" "C49678" (id 4) (at 119.38 76.2 0)
       (effects (font (size 1.27 1.27)) hide)
     )
@@
       (effects (font (size 1.27 1.27)) hide)
     )
+    (property "JLCPCB BOM" "0" (id 4) (at 191.77 99.06 0)
+      (effects (font (size 1.27 1.27)) hide)
+    )
     (pin "1")
     (pin "2")
@@
     )
     (property "Datasheet" "~" (id 3) (at 191.77 127 0)
+      (effects (font (size 1.27 1.27)) hide)
+    )
+    (property "JLCPCB BOM" "0" (id 4) (at 191.77 127 0)
       (effects (font (size 1.27 1.27)) hide)
     )
@@
       (effects (font (size 1.27 1.27)) hide)
     )
+    (property "LCSC Part" "C14909" (id 4) (at 114.3 106.68 0)
+      (effects (font (size 1.27 1.27)) hide)
+    )
